Commit message: Update urdf

File: zb320_description/urdf/model.urdf (robot description, URDF)
Before this commit: robot zb320, 5 links, 4 joints
Links:
- link base_link: mass None -> 1.4110802987401645
- link link_1_1: mass None -> 2.152080592427195
- link link_2_1: mass None -> 0.48368669197035047
- link link_3_1: mass None -> 0.5032706604395567
- link link_4_1: mass None -> 0.12489833913220899
